Commit message: implementing robots orientation

File: universal_robots/UR5e.urdf (robot description, URDF)
Before this commit: robot UR5e, 19 links, 18 joints
Links:
- removed link ROBOTIQ 3f Gripper
- added link ROBOTIQ_3f_Gripper; collision box size=0.126 0.093 0.13; collision cylinder length=0.05 radius=0.023
Joints:
- removed joint wrist_3_link_ROBOTIQ 3f Gripper_joint
- added joint wrist_3_link_ROBOTIQ_3f_Gripper_joint: type fixed, parent wrist_3_link, child ROBOTIQ 3f Gripper, origin xyz=0 0.14 0 rpy=0 0 0
