Commit message: gripper: grasping, releasing

File: UR5e_2.urdf (robot description, URDF)
Before this commit: robot UR5e, 20 links, 19 joints
Joints:
- joint elbow_joint: origin xyz=0 -0.131 0.425 rpy=0 1.570028 0 -> xyz=0 -0.131 0.425 rpy=0 1.569823 0
- joint finger_2_joint_1: origin xyz=0.02 0 0 rpy=0 0 0.000005 -> xyz=0.02 0 0 rpy=0 0 0.000006
- joint palm_finger_1_joint: origin xyz=-0.0455 0.0214 0.036 rpy=3.141592 0.000006 1.571593 -> xyz=-0.0455 0.0214 0.036 rpy=3.141592 0.000005 1.571593
- joint palm_finger_2_joint: origin xyz=-0.0455 0.0214 -0.036 rpy=3.141592 0.000004 1.571593 -> xyz=-0.0455 0.0214 -0.036 rpy=3.141592 0.000009 1.571593
- joint shoulder_lift_joint: origin xyz=0 0.138 0 rpy=0 0.000824 0 -> xyz=0 0.138 0 rpy=0 0.00104 0
- joint shoulder_pan_joint: origin xyz=0 0 0.163 rpy=0 0 -0.000053 -> xyz=0 0 0.163 rpy=0 0 -0.000052
- joint wrist_1_joint: origin xyz=0 0 0.392 rpy=0 0.0008 0 -> xyz=0 0 0.392 rpy=0 0.001052 0
- joint wrist_2_joint: origin xyz=0 0.127 0 rpy=0 0 -1.57 -> xyz=0 0.127 0 rpy=0 0 -1.569708
- joint wrist_3_joint: origin xyz=0 0 0.1 rpy=0 0.000001 0 -> xyz=0 0 0.1 rpy=0 -0.000001 0

Commit message: issue with wrist 2/ end effector: grid_search

File: UR5e_2.urdf (robot description, URDF)
Before this commit: robot UR5e, 20 links, 19 joints
Joints:
- joint finger_1_joint_1: origin xyz=0.02 0 0 rpy=0 0 0.000005 -> xyz=0.02 0 0 rpy=0 0 0.000004
- joint finger_2_joint_1: origin xyz=0.02 0 0 rpy=0 0 0.000007 -> xyz=0.02 0 0 rpy=0 0 0.000006
- joint palm_finger_1_joint: origin xyz=-0.0455 0.0214 0.036 rpy=3.141592 0.000005 1.571593 -> xyz=-0.0455 0.0214 0.036 rpy=3.141592 -0.000021 1.571593
- joint palm_finger_2_joint: origin xyz=-0.0455 0.0214 -0.036 rpy=3.141592 0.000008 1.571593 -> xyz=-0.0455 0.0214 -0.036 rpy=3.141592 0.000009 1.571593
- joint shoulder_lift_joint: origin xyz=0 0.138 0 rpy=0 0.001037 0 -> xyz=0 0.138 0 rpy=0 0.001042 0
- joint wrist_3_link_CAM_joint: origin xyz=0 0.18 0 rpy=-1.570796 0 0.000004 -> xyz=0 0.153473 -0.006378 rpy=0.000004 -0.261798 -0.000002
