Commit message: Final Grid_search method

File: UR5e.urdf (robot description, URDF)
Before this commit: robot UR5e, 20 links, 19 joints
Links:
- removed link ROBOTIQ 3f Gripper
- removed link camera
- removed link finger_1_link_0
- removed link finger_1_link_1
- removed link finger_1_link_2
- removed link finger_1_link_3
- removed link finger_2_link_0
- removed link finger_2_link_1
- removed link finger_2_link_2
- removed link finger_2_link_3
- removed link finger_middle_link_1
- removed link finger_middle_link_2
- removed link finger_middle_link_3
- added link CAM
Joints:
- removed joint finger_1_joint_1
- removed joint finger_1_joint_2
- removed joint finger_1_joint_3
- removed joint finger_2_joint_1
- removed joint finger_2_joint_2
- removed joint finger_2_joint_3
- removed joint finger_middle_joint_1
- removed joint finger_middle_joint_2
- removed joint finger_middle_joint_3
- removed joint palm_finger_1_joint
- removed joint palm_finger_2_joint
- removed joint wrist_3_link_ROBOTIQ 3f Gripper_joint
- removed joint wrist_3_link_camera_joint
