Commit message: orientation completed/ grasp and release

File: UR5e_1.urdf (robot description, URDF)
Before this commit: robot UR5e, 20 links, 19 joints
Links:
- removed link camera
- added link CAM
Joints:
- removed joint wrist_3_link_camera_joint
- added joint wrist_3_link_CAM_joint: type fixed, parent wrist_3_link, child CAM, origin xyz=0 0.18 0 rpy=-1.570796 0 0.000004

File: UR5e_2.urdf (robot description, URDF)
Before this commit: robot UR5e, 20 links, 19 joints
Links:
- removed link camera
- added link CAM
Joints:
- removed joint wrist_3_link_camera_joint
- added joint wrist_3_link_CAM_joint: type fixed, parent wrist_3_link, child CAM, origin xyz=0 0.18 0 rpy=-1.570796 0 0.000004
- joint finger_1_joint_1: origin xyz=0.02 0 0 rpy=0 0 0.000004 -> xyz=0.02 0 0 rpy=0 0 0.000005
- joint finger_2_joint_1: origin xyz=0.02 0 0 rpy=0 0 0.000006 -> xyz=0.02 0 0 rpy=0 0 0.000007
- joint palm_finger_2_joint: origin xyz=-0.0455 0.0214 -0.036 rpy=3.141592 0.000009 1.571593 -> xyz=-0.0455 0.0214 -0.036 rpy=3.141592 0.000008 1.571593
- joint shoulder_lift_joint: origin xyz=0 0.138 0 rpy=0 0.00104 0 -> xyz=0 0.138 0 rpy=0 0.001037 0
- joint shoulder_pan_joint: origin xyz=0 0 0.163 rpy=0 0 -0.000052 -> xyz=0 0 0.163 rpy=0 0 0.000053
- joint wrist_1_joint: origin xyz=0 0 0.392 rpy=0 0.001052 0 -> xyz=0 0 0.392 rpy=0 0.001005 0
- joint wrist_2_joint: origin xyz=0 0.127 0 rpy=0 0 -1.569708 -> xyz=0 0.127 0 rpy=0 0 -1.569795
- joint wrist_3_joint: origin xyz=0 0 0.1 rpy=0 -0.000001 0 -> xyz=0 0 0.1 rpy=0 0.000001 0

Commit message: get Image/ object Detection

File: UR5e_1.urdf (robot description, URDF)
Before this commit: robot UR5e, 20 links, 19 joints
Links:
- added link DISTANCESENSOR
Joints:
- added joint wrist_3_link_DISTANCESENSOR_joint: type fixed, parent wrist_3_link, child DISTANCESENSOR, origin xyz=0 0.21 0 rpy=0 0 0

Commit message: rotational search strategy

File: UR5e_1.urdf (robot description, URDF)
Before this commit: robot UR5e, 21 links, 20 joints
Links:
- removed link DISTANCESENSOR
Joints:
- removed joint wrist_3_link_DISTANCESENSOR_joint

Commit message: continuation of grid_search: incomplete

File: UR5e_1.urdf (robot description, URDF)
Before this commit: robot UR5e, 20 links, 19 joints
Joints:
- joint wrist_3_link_CAM_joint: origin xyz=0 0.18 0 rpy=-1.570796 0 0.000004 -> xyz=0 0.153473 -0.006378 rpy=0.000004 -0.261798 -0.000002

Commit message: Minor modifications

File: UR5e_1.urdf (robot description, URDF)
Before this commit: robot UR5e, 21 links, 20 joints
Links:
- removed link ROBOTIQ_3f_Gripper
- removed link rubber duck
- added link ROBOTIQ 3f Gripper; collision box size=0.126 0.093 0.13; collision cylinder length=0.05 radius=0.023
Joints:
- removed joint wrist_3_link_ROBOTIQ_3f_Gripper_joint
- removed joint wrist_3_link_rubber duck_joint
- added joint wrist_3_link_ROBOTIQ 3f Gripper_joint: type fixed, parent wrist_3_link, child ROBOTIQ 3f Gripper, origin xyz=0 0.14 0 rpy=0 0 0
- joint elbow_joint: origin xyz=0 -0.131 0.425 rpy=0 0.966795 0 -> xyz=0 -0.131 0.425 rpy=0 0 0
- joint finger_1_joint_1: origin xyz=0.02 0 0 rpy=0 0 0.000044 -> xyz=0.02 0 0 rpy=0 0 0
- joint finger_2_joint_1: origin xyz=0.02 0 0 rpy=0 0 0.000027 -> xyz=0.02 0 0 rpy=0 0 0
- joint finger_middle_joint_1: parent ROBOTIQ_3f_Gripper -> ROBOTIQ 3f Gripper
- joint palm_finger_1_joint: origin xyz=-0.0455 0.0214 0.036 rpy=3.141592 -0.000021 1.571593 -> xyz=-0.0455 0.0214 0.036 rpy=3.141592 -0.000008 1.571593; parent ROBOTIQ_3f_Gripper -> ROBOTIQ 3f Gripper
- joint palm_finger_2_joint: origin xyz=-0.0455 0.0214 -0.036 rpy=3.141592 -0.000017 1.571593 -> xyz=-0.0455 0.0214 -0.036 rpy=3.141592 -0.000008 1.571593; parent ROBOTIQ_3f_Gripper -> ROBOTIQ 3f Gripper
- joint shoulder_lift_joint: origin xyz=0 0.138 0 rpy=0 0.729265 0 -> xyz=0 0.138 0 rpy=0 1.570796 0
- joint shoulder_pan_joint: origin xyz=0 0 0.163 rpy=0 0 -0.097213 -> xyz=0 0 0.163 rpy=0 0 0
- joint wrist_1_joint: origin xyz=0 0 0.392 rpy=0 -1.444978 0 -> xyz=0 0 0.392 rpy=0 1.570796 0
- joint wrist_2_joint: origin xyz=0 0.127 0 rpy=0 0 -0.897061 -> xyz=0 0.127 0 rpy=0 0 0
- joint wrist_3_joint: axis 0.000104 1 0.000001 -> 0 1 0; origin xyz=0 0 0.1 rpy=0.000281 1.21761 0.0003 -> xyz=0 0 0.1 rpy=0 0 0
- joint wrist_3_link_camera_joint: origin xyz=0.008619 0.186471 0.006962 rpy=-1.570796 -0.261801 0.261803 -> xyz=0 0.1 0 rpy=-1.570796 0 -1.570796

File: UR5e_2.urdf (robot description, URDF)
Before this commit: robot UR5e, 19 links, 18 joints
Links:
- removed link ROBOTIQ_3f_Gripper
- added link ROBOTIQ 3f Gripper; collision box size=0.126 0.093 0.13; collision cylinder length=0.05 radius=0.023
- added link camera
Joints:
- removed joint wrist_3_link_ROBOTIQ_3f_Gripper_joint
- added joint wrist_3_link_ROBOTIQ 3f Gripper_joint: type fixed, parent wrist_3_link, child ROBOTIQ 3f Gripper, origin xyz=0 0.14 0 rpy=0 0 0
- added joint wrist_3_link_camera_joint: type fixed, parent wrist_3_link, child camera, origin xyz=0 0.1 0 rpy=-1.570796 0 -1.570796
- joint elbow_joint: origin xyz=0 -0.131 0.425 rpy=0 0.928148 0 -> xyz=0 -0.131 0.425 rpy=0 1.570028 0
- joint finger_1_joint_1: origin xyz=0.02 0 0 rpy=0 0 0.000019 -> xyz=0.02 0 0 rpy=0 0 0.000004
- joint finger_2_joint_1: origin xyz=0.02 0 0 rpy=0 0 0.000001 -> xyz=0.02 0 0 rpy=0 0 0.000005
- joint palm_finger_1_joint: origin xyz=-0.0455 0.0214 0.036 rpy=3.141592 0.000008 1.571593 -> xyz=-0.0455 0.0214 0.036 rpy=3.141592 0.000006 1.571593
- joint palm_finger_2_joint: origin xyz=-0.0455 0.0214 -0.036 rpy=3.141592 0.000012 1.571593 -> xyz=-0.0455 0.0214 -0.036 rpy=3.141592 0.000004 1.571593
- joint shoulder_lift_joint: origin xyz=0 0.138 0 rpy=0 0.647298 0 -> xyz=0 0.138 0 rpy=0 0.000824 0
- joint shoulder_pan_joint: origin xyz=0 0 0.163 rpy=0 0 0.884085 -> xyz=0 0 0.163 rpy=0 0 -0.000053
- joint wrist_1_joint: origin xyz=0 0 0.392 rpy=0 0.642915 0 -> xyz=0 0 0.392 rpy=0 0.0008 0
- joint wrist_2_joint: origin xyz=0 0.127 0 rpy=0 0 -0.927503 -> xyz=0 0.127 0 rpy=0 0 -1.57
